File: PCB/TestPCB/TestChildBoardA.kicad_pcb (KiCad board)
At the start: 2 copper layers, 63.4 x 100.1 mm, 19 parts, among them M2 Screw MountingHole_2.2mm_M2

Commit message: Move configurations
Parts:
- added REFFC: Amphenol_F32R-1A7x1-11010_1x10-1MP_P0.5mm_Horizontal, Connector_FFC-FPC:Amphenol_F32R-1A7x1-11010_1x10-1MP_P0.5mm_Horizontal, F.Cu at (87.4, 25.1)
- moved M2 Screw 21.6 mm to (71.9, 19.3)
- moved M2 Screw 0.57 mm to (18.8, 30.5)
Routing:
- net TP: track 0.00 -> 170.5 mm, vias 0 -> 8
- net GND: track 50.1 -> 81.6 mm
- added copper zone on B.Cu, net GND
Other:
- board size 63.4 x 100.1 mm -> 61.2 x 100.1 mm

Commit message: Test PCB Finished
Parts:
- removed C.1μ, CMOD2.2nF: C_0201_0603Metric, Capacitor_SMD:C_0201_0603Metric
- removed C.1μ, C1μ: C_0402_1005Metric, Capacitor_SMD:C_0402_1005Metric
- removed CY8CMBR3116 DIP Module Placement: PinSocket_1x12_P2.54mm_Vertical, Connector_PinSocket_2.54mm:PinSocket_1x12_P2.54mm_Vertical
- removed Connection: PinHeader_1x04_P2.54mm_Vertical, Connector_PinHeader_2.54mm:PinHeader_1x04_P2.54mm_Vertical
- removed R4.7k (x2): R_0402_1005Metric, Resistor_SMD:R_0402_1005Metric
- removed R560 (x8): C_0603_1608Metric, Capacitor_SMD:C_0603_1608Metric
- removed the REF** at (25.9, 27.9)
- added REF**: PinHeader_2x09_P1.27mm_Horizontal, Connector_PinHeader_1.27mm:PinHeader_2x09_P1.27mm_Horizontal, F.Cu at (75.3, 14.6)
- added REF**: PinSocket_2x09_P1.27mm_Horizontal, Connector_PinSocket_1.27mm:PinSocket_2x09_P1.27mm_Horizontal, F.Cu at (22.9, 14.6)
- moved REFFC 68.2 mm to (19.7, 33.8), turned to -90 degrees
- moved M2 Screw 19.0 mm to (32.0, 16.9)
- moved M2 Screw 13.7 mm to (72.0, 33.0)
Connections:
- REFFC pad 1: (no net) -> GND
- REFFC pad 10: (no net) -> GND
- REFFC pad 2: (no net) -> GND
- REFFC pad 3: (no net) -> TP
- REFFC pad 4: (no net) -> GND
- REFFC pad 5: (no net) -> TP
- REFFC pad 6: (no net) -> GND
- REFFC pad 7: (no net) -> TP
- REFFC pad 8: (no net) -> GND
- REFFC pad 9: (no net) -> TP
Routing:
- net TP: track 170.5 -> 513.3 mm, vias 8 -> 12
- net GND: track 81.6 -> 209.9 mm, vias 0 -> 6
- net I²C: track 42.8 -> 0.00 mm, vias 2 -> 0
- net VCC: track 33.2 -> 0.00 mm
- net R-CS: track 19.3 -> 0.00 mm
- net CMOD: track 2.29 -> 0.00 mm
Other:
- board text added: "A"
- board text added: "CS0"
- board text added: "CS11"
- board text added: "CS3"
- board text added: "CS4"
- board text added: "CS7"
- board text added: "CS8"
- board text removed: "1.8~5.5V"
- board text removed: "CS0 CS1 CS2 CS3 CMOD VCC VDD VSS CS15 CS14 CS13 CS12"
- board text removed: "GND"
- board text removed: "SCL"
- board text removed: "SDA"
- board text removed: "VCC"
- board text removed: "XRES' HI' SCL SDA CS4 CS5 CS6 CS7 CS8 CS9 CS10 CS11"
