File: PCB/CY8CMBR3116_PCB/CY8CMBR3116_PCB.kicad_pcb (KiCad board)
At the start: 2 copper layers, 16.3 x 31.5 mm, 3 parts

Commit message: Start making final PCBs
Parts:
- CY8CMBR3116: footprint Package_DFN_QFN:QFN-24-1EP_4x4mm_P0.5mm_EP2.6x2.6mm -> Package_DFN_QFN:QFN-24-1EP_4x4mm_P0.5mm_EP2.65x2.65mm_ThermalVias
Routing:
- net default: vias 1 -> 0
