File: PCB/FormalPCB/Motherboard.kicad_pcb (KiCad board)
At the start: 2 copper layers, 100 x 100 mm, 55 parts, among them M2 Screw MountingHole_2.2mm_M2

Commit message: PCB Large update & ready for LED debug board
Parts:
- removed 1kΩ (x22): R_0402_1005Metric, Resistor_SMD:R_0402_1005Metric
- removed 74HC595 (x3): SOIC-16_3.9x9.9mm_P1.27mm, Package_SO:SOIC-16_3.9x9.9mm_P1.27mm
- removed BarGraph10+ (x2), BarGraph10- (x2): PinHeader_1x10_P2.54mm_Vertical, Connector_PinHeader_2.54mm:PinHeader_1x10_P2.54mm_Vertical
- removed BarGraph5+, BarGraph5-: PinHeader_1x05_P2.54mm_Vertical, Connector_PinHeader_2.54mm:PinHeader_1x05_P2.54mm_Vertical
- removed the R560 at (66.6, 22.7)
- removed the R560 at (66.7, 17.6)
- removed the R560 at (66.6, 25.2)
- removed the R560 at (66.7, 20.1)
- added M2 Screw: MountingHole_2.2mm_M2, MountingHole:MountingHole_2.2mm_M2, F.Cu at (52.5, 26.9)
- added R560: R_0603_1608Metric_Pad0.98x0.95mm_HandSolder, Resistor_SMD:R_0603_1608Metric_Pad0.98x0.95mm_HandSolder, F.Cu at (18.3, 41.9)
- added R560: R_0603_1608Metric_Pad0.98x0.95mm_HandSolder, Resistor_SMD:R_0603_1608Metric_Pad0.98x0.95mm_HandSolder, F.Cu at (42.9, 45.7)
- added R560: R_0603_1608Metric_Pad0.98x0.95mm_HandSolder, Resistor_SMD:R_0603_1608Metric_Pad0.98x0.95mm_HandSolder, F.Cu at (18.3, 35.8)
- added R560: R_0603_1608Metric_Pad0.98x0.95mm_HandSolder, Resistor_SMD:R_0603_1608Metric_Pad0.98x0.95mm_HandSolder, F.Cu at (18.3, 43.4)
- added R560: R_0603_1608Metric_Pad0.98x0.95mm_HandSolder, Resistor_SMD:R_0603_1608Metric_Pad0.98x0.95mm_HandSolder, F.Cu at (18.3, 45.0)
- added R560: R_0603_1608Metric_Pad0.98x0.95mm_HandSolder, Resistor_SMD:R_0603_1608Metric_Pad0.98x0.95mm_HandSolder, F.Cu at (18.3, 40.4)
- added R560: R_0603_1608Metric_Pad0.98x0.95mm_HandSolder, Resistor_SMD:R_0603_1608Metric_Pad0.98x0.95mm_HandSolder, F.Cu at (18.3, 38.9)
- added R560: R_0603_1608Metric_Pad0.98x0.95mm_HandSolder, Resistor_SMD:R_0603_1608Metric_Pad0.98x0.95mm_HandSolder, F.Cu at (42.9, 44.1)
- added R560: R_0603_1608Metric_Pad0.98x0.95mm_HandSolder, Resistor_SMD:R_0603_1608Metric_Pad0.98x0.95mm_HandSolder, F.Cu at (18.3, 34.3)
- added R560: R_0603_1608Metric_Pad0.98x0.95mm_HandSolder, Resistor_SMD:R_0603_1608Metric_Pad0.98x0.95mm_HandSolder, F.Cu at (18.3, 37.3)
- REF** (x4): value JST_GH_BM09B-GHS-TBT_1x09-1MP_P1.25mm_Vertical -> JST_GH_SM05B-GHS-TB_1x05-1MP_P1.25mm_Horizontal; footprint Connector_JST:JST_GH_BM09B-GHS-TBT_1x09-1MP_P1.25mm_Vertical -> Connector_JST:JST_GH_SM05B-GHS-TB_1x05-1MP_P1.25mm_Horizontal
- moved M2 Screw 131.3 mm to (9.91, 27.1)
- moved M2 Screw 77.9 mm to (49.4, 13.5)
- moved U? 50.1 mm to (49.4, 13.5), turned to -90 degrees
- moved REF** 29.7 mm to (3.25, 45.7), turned to -90 degrees
- moved REF** 29.5 mm to (58.0, 45.7), turned to 90 degrees
- moved C.1μ 22.8 mm to (28.3, 46.0)
- moved C.1μ 22.8 mm to (26.7, 46.1)
- moved C1μ 22.8 mm to (29.8, 46.0)
- moved R560 22.4 mm to (42.9, 39.6)
- moved R560 22.4 mm to (42.9, 35.0)
- moved R560 22.4 mm to (42.9, 36.5)
- moved R560 22.4 mm to (42.9, 38.0)
- moved R560 22.4 mm to (42.9, 42.6)
- moved R560 22.4 mm to (42.9, 41.1)
- moved C2.2nF 21.2 mm to (25.9, 42.3)
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Connections:
- REF** pad 3: GND -> TP (x4)
- REF** pad 5: GND -> TP (x2)
- REF** pad 1: GND -> TP (x2)
- U? pad 11: (no net) -> 595CLK
- U? pad 12: (no net) -> 595Din
- U? pad 13: (no net) -> 595latch
- U? pad 4: 595Din -> (no net)
- U? pad 6: 595latch -> (no net)
- U? pad 7: 595CLK -> (no net)
Routing:
- net R-CS: track 0.00 -> 218.8 mm
- net TP: track 30.7 -> 212.0 mm
- net 595Output: track 130.9 -> 0.00 mm
- net 595Din: track 103.5 -> 2.92 mm, vias 2 -> 0
- net R-LED: track 82.4 -> 0.00 mm
- net I²C: track 0.03 -> 75.3 mm
- net VCC: track 39.6 -> 99.2 mm, vias 0 -> 3
- net GND: track 156.6 -> 167.6 mm, vias 6 -> 9
- net 595latch: track 0.00 -> 2.92 mm
- net 595CLK: track 0.00 -> 2.92 mm
Other:
- board size 100 x 100 mm -> 61.3 x 51.1 mm
- board text added: "CS0 CS1 CS2 CS3"
- board text added: "CS15 CS14 CS13 CS12"
- board text added: "CS4 CS5 CS6 CS7"
- board text added: "CS8 CS9 CS10 CS11"
- board text added: "GP10"
- board text added: "GP11"
- board text added: "GP12"
- board text removed: "CS0"
- board text removed: "CS1"
- board text removed: "CS10"
- board text removed: "CS11"
- board text removed: "CS12"
- board text removed: "CS13"
- board text removed: "CS14"
- board text removed: "CS15"
- board text removed: "CS2"
- board text removed: "CS3"
- board text removed: "CS4"
- board text removed: "CS5"
- board text removed: "CS6"
- board text removed: "CS7"
- board text removed: "CS8"
- board text removed: "CS9"
